File: src/HardwareDesign/PCIe-1x-Toolcard.brd (EAGLE design)
At the start: 167.8 x 69.1 mm, 147 parts, among them IC1 TUSB7340RKMR, IC2 24LC01BT-I/OT, IC3 TPS2560DRCR, IC4 TPS2560DRCR, IC5 TPS74401RGWT, IC6 TPS5450DDAR, J1 JUMPER-NO, J2 JUMPER-3, J3 JUMPER-NO, J4 692141030100, J5 692141030100, Y1 48MHz

Commit message: Add JLC06161H-3313A 6-layer stackup configuration with detailed specifications
- Introduced a new XML file for the JLC06161H-3313A PCB stackup.
- Included comprehensive descriptions of layer stackup, materials, and controlled impedance configurations.
- Defined various manufacturing parameters such as copper weights, isolation thicknesses, and pad dimensions.
- Specified controlled impedance configurations for different signal layers.
Parts:
- removed D11, D13: Green, ds_LED:LED-0603
- removed D12: MBRS540T3G, diode:SMC
- removed D2, D3, D4: Red, ds_LED:LED-0603
- removed D5, D6, D7: (no value), ds_ic_peripherals:USON
- removed FB1: (no value), ds_passive:0603
- removed J5: 692141030100, Wurth_Connectors_WR-USB:692141030100
- removed Y1: 48MHz, Wurth_Quartz Crystals & Oscillators_WE-XTAL:WE-XTAL_CFPX-180
- added !PERST, !REQ, !RST, !SMI, AUX3: TPB1,27, testpad:B1,27
- added 1V8, 2V5, 3V3, DBGG, PGOOD3, PGOOD5, UARG: Green, ds_LED:LED-0603
- added C100, C102, C106, C107, C108, C109, C110, C111, C112, C113, C114, C115, C116, C117, C118, C119, C120, C121, C122, C123, C124, C129, C130, C131, C133, C134, C87, C88, C89, C90, C91, C92, C95, C96, C97, C98: 100nF 25V, ds_capacitors:0201
- added C101, C103: 10uF 16V, ds_capacitors:0603
- added C104, C105: 1uF 16V, ds_capacitors:0201
- added C125, C126, C93, C94, C99: 4.7uF 25V, ds_capacitors:0402
- added C127, C128: 12pF 50V, ds_capacitors:0201
- added C132, C135: 10uF 50V, ds_capacitors:0805
- added C86: 27pF 50V, ds_capacitors:0201
- added DBGY, UARY: Yellow, ds_LED:LED-0603
- added G2R, PORT1, PORT2, PORT3, PORT4: Red, ds_LED:LED-0603
- added IC10, IC7: SN74LVC541ARGYR, ds_ic_logic:QFN50P350X450X100-25T305X205N
- added IC11: FT4232HL, ds_ic_peripherals:LQFP64-10X10
- added IC12: 93LC56BT-I/OT, ds_ic_memory:SOT95P280X145-6N
- added IC13, IC25: MIC5504-3.3YM5, ds_ic_vreg:SOT23-5
- added IC14: LMV611MFX/NOPB, ds_ic_opa:SOT23-5
- added IC15, IC16, IC17: TXS0108ERGYR, ds_ic_peripherals:VQFN24
- added IC18, IC19, IC20: TLV3501AIDBVR, ds_ic_opa:SOT95P280X145-6N
- added IC21: RP2040, ds_ic_mcu:QFN56
- added IC22: (no value), ds_ic_memory:SON127P600X500X75-8N
- added IC23, IC24: 74AUP1T17GWH, ds_ic_logic:SOT353-1
- added IC8: CAT24C256HU4IGT3, ds_ic_memory:SON50P300X200X50-9T130X140N
- added IC9: CY7C68013A-56LTXC, ds_ic_mcu:QFN50P800X800X100-57T665
- added J7: JUMPER-NO, ds_passive:J-0402-NO
- added JTAG: 62701021721, Wurth_Connectors_WR-BHD:62701021721
- added LA: 62702021721, Wurth_Connectors_WR-BHD:62702021721
- added R35, R38, R39: 10K 1%, ds_resistor:0402
- added R36, R45, R47, R65: 10K 1%, ds_resistor:0201
- added R37, R41, R42: 100K 1%, ds_resistor:0201
- added R40: 15K 1%, ds_resistor:0201
- added R43, R44, R48: 1K 1%, ds_resistor:0603
- added R46: 7.87K 1%, ds_resistor:0201
- added R49: 4.3K 1%, ds_resistor:0201
- added R50, R53: 1K 1%, ds_resistor:0201
- added R51, R52: 27R 1%, ds_resistor:0201
- added R54, R55, R56, R57, R58: 1K 1%, ds_resistor:0402
- added R59, R60, R61, R62, R63, R64: 100R 1%, ds_resistor:0201
- added RN1, RN10, RN2, RN3, RN4, RN7, RN8, RN9: 100R 1%, ds_resistor:0603X4-1206
- added RN11, RN12, RN5, RN6: 100K 1%, ds_resistor:0603X4-1206
- added RPDBUG, RPUART: SM03B-SRSS-TB, ds_con:SM03B-SRSS-TB
- added SW1, SW2: B3U-1000P, ds_passive:B3U-1000P
- added T1, T2: (no value), ds_active:SOT23
- added UART1, UART2: 62731020621, Wurth_Connectors_WR-BHD:62731020621
- added X1, X2: 24MHz, Wurth_Quartz Crystals & Oscillators_WE-XTAL:WE-XTAL_CFPX-180
- added X3, X4: 12MHz, Wurth_Quartz Crystals & Oscillators_WE-XTAL:WE-XTAL_CFPX-180
- C1, C13, C2, C3, C4, C5: value 100nF 16V -> 100nF 25V; device ds_capacitors:0201 -> ds_capacitors:0402
- C10: value 100nF 16V -> 1nF; device ds_capacitors:0201 -> ds_passive:C0402
- C11, C12, C6, C80, C9: value 100nF 16V -> 10uF 50V; device ds_capacitors:0201 -> ds_capacitors:0805
- C14, C15, C16: value 10nF 16V -> 100nF 25V; device ds_capacitors:0201 -> ds_capacitors:0402
- C21: value 22uF 16V -> 10nF 16V; device ds_capacitors:0805 -> ds_capacitors:0201
- C23: value 10nF 16V -> 100nF 16V
- C26, C28, C30, C32, C34, C35, C36, C39: value 100nF 16V -> 10nF 16V
- C29: value 22uF 16V -> 100nF 16V; device ds_capacitors:0805 -> ds_capacitors:0201
- C37, C38: value 10uF 50V -> 10nF 16V; device ds_capacitors:0805 -> ds_capacitors:0201
- C42, C65: value 100nF 16V -> 1uF 16V
- C43: value 100nF 16V -> 8pF 50V
- C44: value 10uF 50V -> 8pF 50V; device ds_capacitors:0805 -> ds_capacitors:0201
- C45: value 10uF 50V -> 22uF 25V
- C46: value 100nF 25V -> 10uF 16V; device ds_capacitors:0402 -> ds_capacitors:0805
- C47: value 100nF 25V -> 10nF 50V; device ds_capacitors:0402 -> ds_capacitors:0805
- C48: value 100nF 25V -> 10nF 16V; device ds_capacitors:0402 -> ds_capacitors:0201
- C49: value 100nF 25V -> DNI; device ds_capacitors:0402 -> ds_capacitors:0201
- C50: value 1nF -> 10nF 25V; device ds_passive:C0402 -> ds_capacitors:0402
- C51: value 18pF 25V -> 10nF 50V; device ds_capacitors:0201 -> ds_capacitors:0805
- C52: value 18pF 25V -> 330uF 25V; device ds_capacitors:0201 -> ds_capacitors:6.3X7.7(DXL)
- C53: value 100nF 16V -> 22uF 16V; device ds_capacitors:0201 -> ds_capacitors:0805
- C56, C58, C61: value 150uF 35V -> 100nF 16V; device ds_capacitors:6.3X5.5(DXL) -> ds_capacitors:0201
- C59, C60, C64: value 100nF 16V -> 150uF 35V; device ds_capacitors:0201 -> ds_capacitors:6.3X5.5(DXL)
- C66, C74: value 100nF 16V -> 100nF 25V; device ds_capacitors:0603 -> ds_capacitors:0201
- C67: value 1nF 16V -> 100nF 25V; device ds_capacitors:0402 -> ds_capacitors:0201
- C68, C69, C72, C73, C77: value 100nF 16V -> 100nF 25V
- C70: value 10nF 16V -> 100nF 25V
- C71: value DNI -> 100nF 25V
- C75: value 1nF 16V -> 12pF 50V; device ds_capacitors:0402 -> ds_capacitors:0201
- C76: value 100nF 16V -> 12pF 50V
- C78: value 10uF 16V -> 100nF 25V; device ds_capacitors:0805 -> ds_capacitors:0201
- C79: value 22uF 16V -> 100nF 25V; device ds_capacitors:0805 -> ds_capacitors:0201
- C81: value 10nF 50V -> 10uF 50V
- C82: value 22uF 25V -> 100nF 25V; device ds_capacitors:0805 -> ds_capacitors:0201
- C83: value 10nF 25V -> 100nF 25V; device ds_capacitors:0402 -> ds_capacitors:0201
- C84: value 10nF 50V -> 100nF 25V; device ds_capacitors:0805 -> ds_capacitors:0402
- C85: value 330uF 25V -> 27pF 50V; device ds_capacitors:6.3X7.7(DXL) -> ds_capacitors:0201
- D1: value Red -> 1SS294; device ds_LED:LED-0603 -> diode:SOT23
- D10: value (none) -> Red; device ds_ic_peripherals:USON -> ds_LED:LED-0603
- D8: value (none) -> 1N4148SOD-123; device ds_ic_peripherals:USON -> adafruit:SOD-123FL
- D9: value (none) -> MBRS540T3G; device ds_ic_peripherals:USON -> diode:SMC
- IC1: value TUSB7340RKMR -> UPD720201K8-701-BAC-A; device ds_ic_peripherals:RKM100_5P5X5P5 -> ds_ic_peripherals:QFN68-8X8
- IC2: value 24LC01BT-I/OT -> TPS5450DDAR; device 52101-101-REV-A_v16:MEMORY-ATMEL_SOT23-5 -> ds_ic_vreg:8-POWERSOIC
- IC3: value TPS2560DRCR -> TPS74401RGWT; device ds_ic_vreg:VSON10-3X3 -> ds_ic_vreg:VQFN20-5X5
- IC5: value TPS74401RGWT -> TPS2560DRCR; device ds_ic_vreg:VQFN20-5X5 -> ds_ic_vreg:VSON10-3X3
- IC6: value TPS5450DDAR -> MIC5504-3.3YM5-TR; device ds_ic_vreg:8-POWERSOIC -> MCU:SOT23-5
- J3: value JUMPER-NO -> JUMPER-3; device ds_passive:J-0402-NO -> ds_passive:JUMPER-3
- J4: value 692141030100 -> 66100511622; device Wurth_Connectors_WR-USB:692141030100 -> Wurth_Connectors_WR-WTB:66100511622
- R1: value 10K 1% -> 0R 1%
- R10: value DNI -> 1.37K 1%
- R11: value DNI -> 4.42K 1%
- R12: value DNI -> 1K 1%; device ds_resistor:0201 -> ds_resistor:0402
- R13, R14: value 0R 1% -> 30.9K 1%
- R15, R16, R5: value 10K 1% -> 1K 1%; device ds_resistor:0201 -> ds_resistor:0402
- R17, R22: value 30.9K 1% -> 1K 1%; device ds_resistor:0201 -> ds_resistor:0402
- R19: value 1K 1% -> 100K 1%; device ds_resistor:0402 -> ds_resistor:0201
- R2: value DNI -> BLM21PG600SN1; device ds_resistor:0201 -> ds_passive:0603
- R20, R21: value 10K 1% -> 3.3K 1%
- R23: value 1K 1% -> 2K 1%; device ds_resistor:0402 -> ds_resistor:0201
- R24, R28: value 1K 1% -> 10K 1%; device ds_resistor:0402 -> ds_resistor:0201
- R25: value 1M 1% -> 10K 1%; device ds_resistor:0402 -> ds_resistor:0201
- R26: value 4.7K 1% -> 10K 1%
- R27: value 1M 1% -> 4.7K 1%; device ds_resistor:0402 -> ds_resistor:0201
- R29: value 10K 1% -> 12K 1%
- R3: value 0R 1% -> 10K 1%
- R30: value 1.87K 1% -> 1K 1%
- R31: value 4.99K 1% -> 4.7K 1%
- R32: value 10K 1% -> 4.7K 1%; device ds_resistor:0402 -> ds_resistor:0201
- R33: value 3.16K 1% -> 10K 1%
- R34: value 1K 1% -> 22K 1%
- R4: value 4.7K 1% -> 1.6K 1%
- R6: value 9.09K 1% -> 4.7K 1%
- R7: value DNI -> 10K 1%; device ds_resistor:0201 -> ds_resistor:0402
- R8: value DNI -> 3.16K 1%; device ds_resistor:0201 -> ds_resistor:0402
- R9: value DNI -> 10K 1%
- moved R13 220.0 mm to (54.8, 54.5), turned to 90 degrees
- moved R18 214.5 mm to (75.0, 32.9)
- moved D10 213.8 mm to (34.0, 34.8), turned to 90 degrees
- moved R16 213.1 mm to (75.0, 30.3)
- moved D1 211.3 mm to (68.0, 16.8), turned to 270 degrees
- moved C73 210.9 mm to (37.6, 29.2), turned to 270 degrees
- moved R24 210.2 mm to (36.1, 10.8), turned to 180 degrees
- moved R34 208.2 mm to (30.3, 23.8), flipped to the bottom, turned to 270 degrees
- moved R28 207.7 mm to (36.4, 24.4), turned to 180 degrees
- moved R29 204.9 mm to (36.2, 19.2), turned to 270 degrees
- moved R15 204.0 mm to (75.0, 35.4)
- moved C63 202.3 mm to (50.5, 59.5), turned to 270 degrees
- moved C72 201.0 mm to (36.8, 29.2), turned to 270 degrees
- moved R23 200.8 mm to (29.9, 10.1), turned to 270 degrees
- moved C61 195.4 mm to (54.6, 55.9)
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Connections:
- removed net LED_1V1: D11.C, R28.1
- removed net N$37: IC1.B14, R4.1
- removed net N$54: IC1.A49, R10.2
- removed net N$55: IC1.B46, R9.2
- removed net N$56: IC1.B47, R8.2
- removed net N$57: IC1.B48, R7.2
- removed net N$59: IC1.A24, R6.1
- removed net PCIE_CAPTX_N: C36.2, PCIE-1X1.A17
- removed net PCIE_CAPTX_P: C35.2, PCIE-1X1.A16
- removed net SHIELD-1: C66.1, C67.1, J4.S3, J4.S4, J5.S3, J5.S4, R25.1
- removed net SHIELD-2: C74.1, C75.1, J4.S1, J4.S2, J5.S1, J5.S2, R27.1
- removed net USB1_CSSTX_N: C64.1, J4.8
- removed net USB1_CSSTX_P: C65.1, J4.9
- removed net USB2_CSSTX_N: C68.1, J5.8
- removed net USB2_CSSTX_P: C69.1, J5.9
- removed net USB3_CSSTX_N: C72.1, J4.17
- removed net USB3_CSSTX_P: C73.1, J4.18
- removed net USB4_CSSTX_N: C76.1, J5.17
- removed net USB4_CSSTX_P: C77.1, J5.18
- new net !CTS1: IC11.41, IC16.15
- new net !CTS1_OUT: IC16.6, UART1.5
- new net !CTS2: IC11.54, IC17.15
- new net !CTS2_OUT: IC17.6, UART2.6
- new net !DCD1: IC11.45, IC16.18
- new net !DCD1_OUT: IC16.3, UART1.10
- new net !DCD2: IC11.58, IC17.18
- new net !DCD2_OUT: IC17.3, UART2.1
- new net !DSR1: IC11.44, IC16.17
- new net !DSR1_OUT: IC16.4, UART1.9
- new net !DSR2: IC11.57, IC17.17
- new net !DSR2_OUT: IC17.4, UART2.2
- new net !DTR1: IC11.43, IC16.16
- new net !DTR1_OUT: IC16.5, UART1.4
- new net !DTR2: IC11.55, IC17.16
- new net !DTR2_OUT: IC17.5, UART2.7
- new net !PECREQ: !REQ.TP, IC1.13
- new net !RI1: IC11.46, IC16.20
- new net !RI1_OUT: IC16.1, UART1.3
- new net !RI2: IC11.59, IC17.20
- new net !RI2_OUT: IC17.1, UART2.8
- new net !RTS1: IC11.40, IC16.14
- new net !RTS1_OUT: IC16.7, UART1.7
- new net !RTS2: IC11.53, IC17.14
- new net !RTS2_OUT: IC17.7, UART2.4
- new net !SMI: !SMI.TP, IC1.1
- new net !SPI_CS: IC1.17
- new net +1V05: C17.1, C18.1, C19.1, C20.1, C21.1, C22.1, C23.1, C24.1, C25.1, C26.1, C27.1, C28.1, C29.1, C53.1, IC1.12, IC1.28, IC1.37, IC1.43, IC1.46, IC1.54, IC1.60, IC1.63, IC1.9, IC3.1, IC3.18, IC3.19, IC3.20, R10.1
- new net +1V8: C95.1, C96.1, C97.1, C98.1, C99.1, IC11.12, IC11.37, IC11.49, IC11.64
- new net +3V3B: C66.1, C67.1, C68.1, C69.1, C70.1, C71.1, C72.1, C73.1, C74.1, C77.1, C78.1, C81.1, C82.1, C83.1, D8.C, IC10.20, IC6.5, IC7.20, IC8.8, IC9.11, IC9.17, IC9.27, IC9.3, IC9.32, IC9.43, IC9.44, IC9.55, IC9.7, R19.1, R20.2, R21.2, RN11.A2, RN11.B2, RN11.C2, RN11.D2, RN12.A2, RN12.B2, RN12.C2, RN12.D2, RN5.A2, RN5.B2, RN5.C2, RN5.D2, RN6.A2, RN6.B2, RN6.C2, RN6.D2
- new net +3V3C: C102.1, C103.1, C109.1, C111.1, C113.1, C84.1, C87.1, C88.1, C89.1, C90.1, C91.1, C92.1, C93.1, C94.1, IC11.20, IC11.31, IC11.4, IC11.42, IC11.50, IC11.56, IC11.9, IC12.6, IC13.5, IC15.19, IC16.19, IC17.19, R24.1, R25.1, R26.1, R31.1, R32.1, R33.1
- new net +3V3D: C117.1, C118.1, C119.1, C120.1, C121.1, C122.1, C125.1, C129.1, C130.1, C131.1, C134.1, C135.1, IC21.1, IC21.10, IC21.22, IC21.33, IC21.42, IC21.43, IC21.44, IC21.48, IC21.49, IC22.8, IC23.5, IC24.5, IC25.5, R65.1
- new net 4232R_RESET: R27.2, R28.1, R30.1
- new net 4232_RESET: IC11.14, R30.2
- new net BOOT: R53.1, SW2.1
- new net BUF_PB0: IC7.18, RN3.A1
- new net BUF_PB1: IC7.17, RN3.B1
- new net BUF_PB2: IC7.16, RN3.C1
- new net BUF_PB3: IC7.15, RN3.D1
- new net BUF_PB4: IC7.14, RN4.A1
- new net BUF_PB5: IC7.13, RN4.B1
- new net BUF_PB6: IC7.12, RN4.C1
- new net BUF_PB7: IC7.11, RN4.D1
- new net BUF_PD0: IC10.18, RN9.A1
- new net BUF_PD1: IC10.17, RN9.B1
- new net BUF_PD2: IC10.16, RN9.C1
- new net BUF_PD3: IC10.15, RN9.D1
- new net BUF_PD4: IC10.14, RN10.A1
- new net BUF_PD5: IC10.13, RN10.B1
- new net BUF_PD6: IC10.12, RN10.C1
- new net BUF_PD7: IC10.11, RN10.D1
- new net CH0: LA.17, RN1.A1
- new net CH1: LA.15, RN1.B1
- new net CH10: LA.8, RN7.C1
- new net CH11: LA.10, RN7.D1
- new net CH12: LA.12, RN8.A1
- new net CH13: LA.14, RN8.B1
- new net CH14: LA.16, RN8.C1
- new net CH15: LA.18, RN8.D1
- new net CH2: LA.13, RN1.C1
- new net CH3: LA.11, RN1.D1
- new net CH4: LA.9, RN2.A1
- new net CH5: LA.7, RN2.B1
- new net CH6: LA.5, RN2.C1
- new net CH7: LA.3, RN2.D1
- new net CH8: LA.4, RN7.A1
- new net CH9: LA.6, RN7.B1
- new net CHI0: IC7.2, RN1.A2, RN5.A1
- new net CHI1: IC7.3, RN1.B2, RN5.B1
- new net CHI10: IC10.4, RN11.C1, RN7.C2
- new net CHI11: IC10.5, RN11.D1, RN7.D2
- new net CHI12: IC10.6, RN12.A1, RN8.A2
- new net CHI13: IC10.7, RN12.B1, RN8.B2
- new net CHI14: IC10.8, RN12.C1, RN8.C2
- new net CHI15: IC10.9, RN12.D1, RN8.D2
- new net CHI2: IC7.4, RN1.C2, RN5.C1
- new net CHI3: IC7.5, RN1.D2, RN5.D1
- new net CHI4: IC7.6, RN2.A2, RN6.A1
- new net CHI5: IC7.7, RN2.B2, RN6.B1
- new net CHI6: IC7.8, RN2.C2, RN6.C1
- new net CHI7: IC7.9, RN2.D2, RN6.D1
- new net CHI8: IC10.2, RN11.A1, RN7.A2
- new net CHI9: IC10.3, RN11.B1, RN7.B2
- new net CLK: R62.2, RPDBUG.1
- new net COMP18_O: IC20.5, R48.1
- new net COMP25_O: IC19.5, R44.1
- new net COMP33_O: IC18.5, R43.1
- new net D25: R35.2, T2.3
- new net D33: R34.2, T1.3
- new net DIO: R63.2, R64.2, RPDBUG.3
- new net EECLK: IC11.62, IC12.4, R26.2
- new net EECS: IC11.63, IC12.5, R24.2
- new net EEDATA: IC11.61, IC12.3, R23.2, R25.2
- new net FT_SCL: IC11.16, IC15.12, R32.2
- new net FT_SCL_OUT: IC15.9
- new net FT_SDA: IC11.17, IC11.18, IC15.13, R31.2
- new net FT_SDA_OUT: IC15.8
- new net GPIO12: IC21.15, R62.1
- new net GPIO13: IC21.16, IC24.4
- new net GPIO14: IC21.17, R63.1
- new net GPIO15: IC21.18, R57.1
- new net GPIO16: IC21.27, R58.1
- new net GPIO2: IC21.4, R54.1
- new net GPIO4: IC21.6, R59.1
- new net GPIO5: IC21.7, IC23.4
- new net GPIO6: IC21.8, R60.1
- new net GPIO7: IC21.9, R55.1
- new net GPIO8: IC21.11, R56.1
- new net ILIM12: IC4.7, R13.1
- new net ILIM34: IC5.7, R14.1
- new net JTAG_TDO: J1.2, PCIE-1X1.A7
- new net KEY: JTAG.7
- new net LA_LED: D10.C, R22.1
- new net LED_3V: PGOOD3.A, R5.2
- new net LED_5V: PGOOD5.A, R12.2
- new net N$11: C128.1, R50.2, X4.3
- new net N$12: 2V5.A, R44.2
- new net N$13: IC21.21, R50.1
- new net N$14: 1V8.A, R48.2
- new net N$15: J7.2, JTAG.1
- new net N$16: G2R.A, R54.2
- new net N$17: DBGG.A, R57.2
- new net N$18: DBGY.A, R58.2
- new net N$19: R56.2, UARY.A
- new net N$20: R55.2, UARG.A
- new net N$21: IC24.2, R64.1
- new net N$24: IC23.2, R61.1
- new net N$8: 3V3.A, R43.2
- new net PA0: IC9.33
- new net PA1: D10.A, IC9.34
- new net PA2: IC9.35
- new net PA3: IC9.36
- new net PA4: IC9.37
- new net PA5: IC9.38
- new net PA6: IC9.39
- new net PA7: IC9.40
- new net PB0: IC9.18, RN3.A2
- new net PB1: IC9.19, RN3.B2
- new net PB2: IC9.20, RN3.C2
- new net PB3: IC9.21, RN3.D2
- new net PB4: IC9.22, RN4.A2
- new net PB5: IC9.23, RN4.B2
- new net PB6: IC9.24, RN4.C2
- new net PB7: IC9.25, RN4.D2
- new net PCIE_CTX_N: C8.2, PCIE-1X1.A17
- new net PCIE_CTX_P: C7.2, PCIE-1X1.A16
- new net PD0: IC9.45, RN9.A2
- new net PD1: IC9.46, RN9.B2
- new net PD2: IC9.47, RN9.C2
- new net PD3: IC9.48, RN9.D2
- new net PD4: IC9.49, RN10.A2
- new net PD5: IC9.50, RN10.B2
- new net PD6: IC9.51, RN10.C2
- new net PD7: IC9.52, RN10.D2
- new net PH: C50.2, D9.C, IC2.8, L1.2
- new net QSPI_SCLK: IC21.52, IC22.6
- new net QSPI_SD0: IC21.53, IC22.5
- new net QSPI_SD1: IC21.55, IC22.2
- new net QSPI_SD2: IC21.54, IC22.3
- new net QSPI_SD3: IC21.51, IC22.7
- new net QSPI_SS: IC21.56, IC22.1, R53.2
- new net RESET: C65.1, D8.A, IC9.42, R19.2
- new net RUN: IC21.26, R65.2, SW1.1
- new net RXD1: IC11.39, IC16.13
- new net RXD1_OUT: IC16.8, UART1.8
- new net RXD2: IC11.52, IC17.13
- new net RXD2_OUT: IC17.8, UART2.3
- new net SPI_MISO: IC1.19
- new net SPI_MOSI: IC1.16
- new net SPI_SCK: IC1.18
- new net SWCLK: IC21.24
- new net SWDIO: IC21.25
- new net TCK/SCK: IC11.26, IC15.16
- new net TCK/SCK_OUT: IC15.5, JTAG.4
- new net TDI/DO: IC11.27, IC15.17
- new net TDI/DO_OUT: IC15.4, JTAG.8
- new net TDO/DI: IC11.28, IC15.18
- new net TDO/DI_OUT: IC15.3, JTAG.6
- new net TMS/CS: IC11.29, IC15.20
- new net TMS/CS_OUT: IC15.1, JTAG.2
- new net TRESET: IC11.30
- new net TRESET_OUT: JTAG.10
- new net TXD1: IC11.38, IC16.12
- new net TXD1_OUT: IC16.9, UART1.6
- new net TXD2: IC11.48, IC17.12
- new net TXD2_OUT: IC17.9, UART2.5
- new net UART1_RX: R60.2, R61.2, RPUART.3
- new net UART1_TX: R59.2, RPUART.1
- new net USB_PID_N: IC21.46, R51.2
- new net USB_PID_P: IC21.47, R52.1
- new net VDIV_BUF: C104.1, IC14.1, R33.2, R34.1, R35.1
- new net VREF_LOGIC: C107.1, C108.1, C110.1, C112.1, IC14.3, IC14.4, IC15.10, IC15.2, IC16.10, IC16.2, IC17.10, IC17.2, IC18.3, IC19.3, IC20.3, J7.1, R37.1, R41.1, R42.1
- new net VSEL_1V8: IC11.23, R39.1, T2.1
- new net VSEL_2V5: IC11.24, R38.1, T1.1
- new net V_COMP18: IC20.1, R47.2, R49.1
- new net V_COMP25: IC19.1, R45.2, R46.1
- new net V_COMP33: IC18.1, R36.2, R40.1
- new net XIN: C75.1, IC9.5, X2.1
- new net XOUT: C76.1, IC9.4, X2.3
- net !GRST: now also !RST.TP, C42.1, C54.1, D1.1, IC1.14, IC3.9, R3.2, R9.2; no longer C80.1, IC1.A15, IC5.9, R29.2
- net !OVERCUR1: now also IC1.26, IC4.10; no longer IC1.A36, IC3.6
- net !OVERCUR2: now also IC1.24, IC4.6; no longer IC1.A37, IC4.10
- net !OVERCUR3: now also IC1.22, IC5.10; no longer IC1.B43, IC3.10
- net !OVERCUR4: now also IC1.20, IC5.6; no longer IC1.B45, IC4.6
- net !PERST: now also !PERST.TP, IC1.2; no longer IC1.A40
- net !PWRON1: now also IC1.27, IC4.4; no longer IC1.B33, IC3.5
- net !PWRON2: now also IC1.25, IC4.5; no longer IC1.B34, IC4.4
- net !PWRON3: now also IC1.23, IC5.4; no longer IC1.A46, IC3.4
- net !PWRON4: now also IC1.21, IC5.5; no longer IC1.A48, IC4.5
- net !WAKE: now also C10.1, IC1.3, R1.2; no longer C50.1, IC1.B35, R3.2
- net !WAKE_R: now also R1.1; no longer R3.1
- net +12V: now also C1.1, C2.1, C3.1, C4.1, C45.1, C47.1, C5.1, C6.1, C9.1, IC2.7; no longer C37.1, C38.1, C39.1, C40.1, C41.1, C42.1, C43.1, C81.1, C82.1, IC6.7
- net +1V1: now also C123.1, C124.1, C126.1, IC21.23, IC21.45, IC21.50; no longer C1.1, C10.1, C11.1, C12.1, C13.1, C14.1, C15.1, C16.1, C17.1, C18.1, C19.1, C2.1, C20.1, C21.1, C3.1, C4.1, C5.1, C6.1, C7.1, C79.1, C8.1, C9.1, IC1.A1, IC1.A12, IC1.A16, IC1.A28, IC1.A31, IC1.A33, IC1.A38, IC1.A4, IC1.A50, IC1.A6, IC1.A9, IC1.B1, IC1.B17, IC1.B19, IC1.B24, IC1.B37, IC1.B40, IC1.B42, IC1.B44, IC5.1, IC5.18, IC5.19, IC5.20, R30.1
- net +3V3: now also C36.1, C38.1, C39.1, C40.1, C41.1, C46.1, D1.3, IC1.15, IC1.29, IC1.40, IC1.49, IC1.57, IC1.66, IC3.10, IC3.5, IC3.6, IC3.7, IC3.8, R2.1, R3.1, R5.1, R6.1; no longer C31.1, C33.1, C53.1, C78.1, D11.A, FB1.1, IC1.A3, IC1.A34, IC1.A39, IC1.A47, IC1.A51, IC2.4, IC5.10, IC5.5, IC5.6, IC5.7, IC5.8, R1.1, R10.1, R11.1, R12.1, R15.1, R16.1, R20.1, R21.1, R26.1, R29.1, R7.1, R8.1
- net +3V3A: now also C31.1, C33.1, C35.1, C37.1, IC1.32, IC1.6, R2.2; no longer C22.1, C23.1, C24.1, C25.1, C26.1, C27.1, C28.1, C29.1, FB1.2, IC1.A19, IC1.A21, IC1.A25, IC1.A44, IC1.B11, IC1.B22, IC1.B26, IC1.B4
- net +3V3_AUX: now also AUX3.TP
- net +5V: now also C51.1, C52.1, C55.1, C56.1, IC5.2, IC5.3, R12.1, R7.1; no longer C54.1, C59.1, C84.1, C85.1, IC3.2, IC3.3, R32.1, R34.1
- net BOOT_5V: now also C50.1, IC2.1; no longer C83.1, IC6.1
- net DS1_VBUS: now also C59.1, C79.1, C80.1, IC4.9, IC6.1, IC6.3, R17.1; no longer C58.1, IC3.8, J4.1, R16.2, R18.1
- net DS2_VBUS: now also C100.1, C101.1, C105.1, C106.1, C114.1, C115.1, C116.1, C63.1, IC13.1, IC13.3, IC14.5, IC18.4, IC19.4, IC20.4, IC4.8, R15.1, R27.1, R36.1, R45.1, R47.1; no longer C60.1, IC4.9, J5.1, R20.2, R24.1
- net DS3_VBUS: now also C132.1, C133.1, C58.1, C60.1, IC25.1, IC25.3, IC5.9, R18.1; no longer C55.1, C56.1, IC3.9, J4.10, R15.2, R19.1
- net DS4_VBUS: now also C64.1, IC5.8, J4.1, R16.1; no longer C63.1, IC4.8, J5.10, R21.2, R23.1
- net EN_1V1: now also C48.1, IC3.11, R6.2; no longer C70.1, IC5.11, R26.2
- net FB_1V1: now also IC3.16, R10.2, R11.1; no longer IC5.16, R30.2, R31.1
- net FB_5V: now also IC2.4, R7.2, R8.1; no longer IC6.4, R32.2, R33.1
- net GND: now also 1V8.C, 2V5.C, 3V3.C, C100.2, C101.2, C102.2, C103.2, C104.2, C105.2, C106.2, C107.2, C108.2, C109.2, C110.2, C111.2, C112.2, C113.2, C114.2, C115.2, C116.2, C117.2, C118.2, C119.2, C120.2, C121.2, C122.2, C123.2, C124.2, C125.2, C126.2, C127.2, C128.2, C129.2, C130.2, C131.2, C132.2, C133.2, C134.2, C135.2, C35.2, C36.2, C64.2, C65.2, C68.2, C69.2, C72.2, C73.2, C76.2, C77.2, C83.2, C86.2, C87.2, C88.2, C89.2, C90.2, C91.2, C92.2, C93.2, C94.2, C95.2, C96.2, C97.2, C98.2, C99.2, D9.A, DBGG.C, DBGY.C, G2R.C, IC1.34, IC1.69, IC10.1, IC10.10, IC10.19, IC10.PAD, IC11.1, IC11.10, IC11.11, IC11.13, IC11.15, IC11.25, IC11.35, IC11.47, IC11.5, IC11.51, IC12.2, IC13.2, IC14.2, IC15.11, IC15.PAD, IC16.11, IC16.PAD, IC17.11, IC17.PAD, IC18.2, IC18.6, IC19.2, IC19.6, IC2.6, IC2.PAD, IC2.V1, IC2.V2, IC2.V3, IC2.V4, IC2.V5, IC2.V6, IC2.V7, IC2.V8, IC20.2, IC20.6, IC21.19, IC21.PAD, IC22.4, IC22.PAD, IC23.3, IC24.3, IC25.2, IC3.12, IC3.21, IC5.1, IC5.PAD, IC6.2, IC7.1, IC7.10, IC7.19, IC7.PAD, IC8.1, IC8.2, IC8.3, IC8.4, IC8.7, IC8.9, IC9.10, IC9.12, IC9.14, IC9.26, IC9.28, IC9.41, IC9.53, IC9.56, IC9.57, IC9.6, J3.2, J4.5, JTAG.3, JTAG.5, JTAG.9, LA.1, LA.19, LA.2, LA.20, PGOOD3.C, PGOOD5.C, PORT1.C, PORT2.C, PORT3.C, PORT4.C, R11.2, R29.2, R37.2, R38.2, R39.2, R40.2, R41.2, R42.2, R46.2, R49.2, R8.2, RPDBUG.2, RPDBUG.S1, RPDBUG.S2, RPUART.2, RPUART.S1, RPUART.S2, SW1.2, SW2.2, T1.2, T2.2, UARG.C, UART1.2, UART2.9, UARY.C, X1.2, X1.4, X2.2, X2.4, X3.2, X3.4, X4.2, X4.4; no longer C50.2, C7.2, C8.2, D1.C, D10.3, D10.8, D12.A, D13.C, D2.C, D3.C, D4.C, D5.3, D5.8, D6.3, D6.8, D7.3, D7.8, D8.3, D8.8, D9.3, D9.8, IC1.B20, IC1.B21, IC1.C1, IC1.C2, IC1.C3, IC1.C4, IC1.PAD, IC1.V, IC1.V_10, IC1.V_12, IC1.V_14, IC1.V_16, IC1.V_18, IC1.V_2, IC1.V_20, IC1.V_22, IC1.V_24, IC1.V_26, IC1.V_28, IC1.V_30, IC1.V_32, IC1.V_34, IC1.V_36, IC1.V_38, IC1.V_4, IC1.V_40, IC1.V_42, IC1.V_44, IC1.V_46, IC1.V_48, IC1.V_6, IC1.V_8, IC2.2, IC2.5, IC3.1, IC3.PAD, IC5.12, IC5.21, IC6.6, IC6.PAD, IC6.V1, IC6.V2, IC6.V3, IC6.V4, IC6.V5, IC6.V6, IC6.V7, IC6.V8, J1.2, J4.13, J4.16, J4.4, J4.7, J5.13, J5.16, J5.4, J5.7, R17.2, R2.2, R25.2, R27.2, R31.2, R33.2, R5.1, Y1.2, Y1.4
- net JTAG_TDITDO: now also J1.1; no longer J3.1
- net LEDDS1: now also PORT2.A, R15.2; no longer D1.A, R18.2
- net LEDDS2: now also PORT3.A, R18.2; no longer D4.A, R24.2
- net LEDDS3: now also PORT1.A, R17.2; no longer D2.A, R19.2
- net LEDDS4: now also PORT4.A, R16.2; no longer D3.A, R23.2
- net N$1: now also IC21.2, J3.1; no longer IC1.A52, J1.1, R1.2, R2.1
- net N$10: now also C86.1, IC11.3, X3.3; no longer C83.2, D12.C, IC6.8, L1.2
- net N$2: now also IC11.6, R29.1; no longer J3.2, PCIE-1X1.A7
- net N$3: now also C85.1, IC11.2, X3.1; no longer IC1.B32, R5.2
- net N$4: now also C43.1, IC1.31, X1.1; no longer C51.1, IC1.A22, Y1.1
- net N$5: now also C44.1, IC1.30, X1.3; no longer C52.1, IC1.A23, Y1.3
- net N$6: now also IC12.1, R23.1; no longer IC3.7, R17.1
- net N$60: now also IC1.33, R4.1; no longer IC1.B23, R6.2
- net N$7: now also IC21.3, J3.3; no longer D13.A, R34.2
- net N$9: now also C127.1, IC21.20, X4.1; no longer IC4.7, R22.1
- net PCIE_3V3: now also C11.1, C12.1, C13.1, C14.1, C15.1, C16.1; no longer C44.1, C45.1, C46.1, C47.1, C48.1, C49.1
- net PCIE_REFCLK_N: now also IC1.4; no longer IC1.B41
- net PCIE_REFCLK_P: now also IC1.5; no longer IC1.A45
- net PCIE_RX_N: now also IC1.11; no longer IC1.A42
- net PCIE_RX_P: now also IC1.10; no longer IC1.B39
- net PCIE_TX_N: now also C8.1, IC1.8; no longer C36.1, IC1.A41
- net PCIE_TX_P: now also C7.1, IC1.7; no longer C35.1, IC1.B38
- net SCL: now also IC8.6, IC9.15, R20.1; no longer IC1.B2, IC2.1, R11.2, R13.1
- net SDA: now also IC8.5, IC9.16, R21.1; no longer IC1.A2, IC2.3, R12.2, R14.1
- net SS: now also C49.1, IC3.15; no longer C71.1, IC5.15
- net USB1_DP_N: now also IC1.42, IC9.9; no longer D5.1, D5.10, IC1.B18, J4.2
- net USB1_DP_P: now also IC1.41, IC9.8; no longer D5.2, D5.9, IC1.A20, J4.3
- net USB1_SSRX_N: now also IC1.39; no longer D5.4, D5.7, IC1.B16, J4.5
- net USB1_SSRX_P: now also IC1.38; no longer D5.5, D5.6, IC1.A18, J4.6
- net USB1_SSTX_N: now also IC1.36; no longer C64.2, D6.1, D6.10, IC1.B15
- net USB1_SSTX_P: now also IC1.35; no longer C65.2, D6.2, D6.9, IC1.A17
- net USB2_DP_N: now also IC1.51, IC11.7; no longer D6.4, D6.7, IC1.A13, J5.2
- net USB2_DP_P: now also IC1.50, IC11.8; no longer D6.5, D6.6, IC1.B12, J5.3
- net USB2_SSRX_N: now also IC1.48; no longer D7.1, D7.10, IC1.A10, J5.5
- net USB2_SSRX_P: now also IC1.47; no longer D7.2, D7.9, IC1.B9, J5.6
- net USB2_SSTX_N: now also IC1.45; no longer C68.2, D7.4, D7.7, IC1.B10
- net USB2_SSTX_P: now also IC1.44; no longer C69.2, D7.5, D7.6, IC1.A11
- net USB3_DP_N: now also IC1.59, R51.1; no longer D8.1, D8.10, IC1.A27, J4.11
- net USB3_DP_P: now also IC1.58, R52.2; no longer D8.2, D8.9, IC1.B25, J4.12
- net USB3_SSRX_N: now also IC1.56; no longer D8.4, D8.7, IC1.A29, J4.14
- net USB3_SSRX_P: now also IC1.55; no longer D8.5, D8.6, IC1.B27, J4.15
- net USB3_SSTX_N: now also IC1.53; no longer C72.2, D9.1, D9.10, IC1.A30
- net USB3_SSTX_P: now also IC1.52; no longer C73.2, D9.2, D9.9, IC1.B28
- net USB4_DP_N: now also IC1.68, J4.2; no longer D9.4, D9.7, IC1.A5, J5.11
- net USB4_DP_P: now also IC1.67, J4.3; no longer D9.5, D9.6, IC1.B5, J5.12
- net USB4_SSRX_N: now also IC1.65; no longer D10.1, D10.10, IC1.A7, J5.14
- net USB4_SSRX_P: now also IC1.64; no longer D10.2, D10.9, IC1.B6, J5.15
- net USB4_SSTX_N: now also IC1.62; no longer C76.2, D10.4, D10.7, IC1.A8
- net USB4_SSTX_P: now also IC1.61; no longer C77.2, D10.5, D10.6, IC1.B7
Routing:
- net GND: track 46.7 -> 431.5 mm, vias 4 -> 382
- net DS2_VBUS: track 0.00 -> 129.5 mm, vias 0 -> 18
- net +3V3B: track 0.00 -> 94.5 mm, vias 0 -> 23
- net DS3_VBUS: track 0.00 -> 81.5 mm, vias 0 -> 25
- net DS1_VBUS: track 0.00 -> 75.7 mm, vias 0 -> 10
- net +12V: track 0.00 -> 72.2 mm, vias 0 -> 14
- net +3V3: track 4.61 -> 69.0 mm, vias 3 -> 29
- net VREF_LOGIC: track 0.00 -> 57.4 mm, vias 0 -> 7
- net +1V05: track 0.00 -> 54.9 mm, vias 0 -> 21
- net USB4_DP_P: track 0.00 -> 47.6 mm, vias 0 -> 1
- net USB4_DP_N: track 0.00 -> 47.6 mm, vias 0 -> 1
- net RUN: track 0.00 -> 47.4 mm, vias 0 -> 2
- net +3V3C: track 0.00 -> 44.9 mm, vias 0 -> 18
- net !OVERCUR2: track 0.00 -> 43.2 mm, vias 0 -> 2
- net USB3_DP_N: track 0.00 -> 42.5 mm, vias 0 -> 2
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- added copper zone on layer 1, net +12V
- added copper zone on layer 16, net +12V
- added copper zone on layer 3, net +12V
- added copper zone on layer 1, net +1V05
- added copper zone on layer 3, net +1V05
- added copper zone on layer 3, net +1V8
- added copper zone on layer 1, net +3V3
- added copper zone on layer 3, net +3V3
- added copper zone on layer 3, net +3V3A
- added copper zone on layer 3, net +3V3B
- added copper zone on layer 3, net +3V3C
- added copper zone on layer 3, net +3V3D
- added copper zone on layer 1, net +5V
- added copper zone on layer 1, net DS1_VBUS
- added copper zone on layer 3, net DS1_VBUS
- added copper zone on layer 1, net DS2_VBUS
- added copper zone on layer 3, net DS2_VBUS
- added copper zone on layer 1, net DS3_VBUS
- added copper zone on layer 16, net DS3_VBUS
- added copper zone on layer 3, net DS3_VBUS
- added copper zone on layer 1, net DS4_VBUS
- added copper zone on layer 16, net DS4_VBUS
- added copper zone on layer 1, net GND
- added copper zone on layer 14, net GND
- added copper zone on layer 15, net GND
- added copper zone on layer 16, net GND
- added copper zone on layer 2, net GND
- added copper zone on layer 1, net PCIE_3V3
- added copper zone on layer 16, net PCIE_3V3
- added copper zone on layer 1, net PH
Other:
- board size 167.8 x 69.1 mm -> 86.7 x 69.1 mm
- board text added: "1"
- board text added: "2"
- board text added: "3"
- board text added: "4"
- board text added: "5"
- board text added: "6"
