File: src/HardwareDesign/PCIe-1x-Toolcard.sch (EAGLE design)
At the start: 147 parts, among them IC1 TUSB7340RKMR, IC2 24LC01BT-I/OT, IC3 TPS2560DRCR, IC4 TPS2560DRCR, IC5 TPS74401RGWT, IC6 TPS5450DDAR, J1 JUMPER-NO, J2 JUMPER-3, J3 JUMPER-NO, J4 692141030100, J5 692141030100, Y1 48MHz

Commit message: Add JLC06161H-3313A 6-layer stackup configuration with detailed specifications
- Introduced a new XML file for the JLC06161H-3313A PCB stackup.
- Included comprehensive descriptions of layer stackup, materials, and controlled impedance configurations.
- Defined various manufacturing parameters such as copper weights, isolation thicknesses, and pad dimensions.
- Specified controlled impedance configurations for different signal layers.
Parts:
- removed D11: Green, ds_LED:LED-GREENLED-0603
- removed D12: MBRS540T3G, diode:DIODE-SMC
- removed D3: Red, ds_LED:LED-REDLED-0603
- removed D5, D6, D7: (no value), ds_ic_peripherals:TPD4EUSB30
- removed FB1: (no value), ds_passive:R0603
- removed J5: 692141030100, Wurth_Connectors_WR-USB:692141030100
- removed Y1: 48MHz, Wurth_Quartz Crystals & Oscillators_WE-XTAL:WE-XTAL_CFPX-180_830108207709
- added !PERST, !REQ, !RST, !SMI, AUX3: TPB1,27, testpad:TPB1,27
- added 1V8, 2V5, 3V3, DBGG, PGOOD3, UARG: Green, ds_LED:LED-GREENLED-0603
- added C100, C102, C106, C107, C108, C109, C110, C111, C112, C113, C114, C115, C116, C117, C118, C119, C120, C121, C122, C123, C124, C129, C130, C131, C133, C134, C87, C88, C89, C90, C91, C92, C95, C96, C97, C98: 100nF 25V, ds_capacitors:100NF-25V-0201
- added C101, C103: 10uF 16V, ds_capacitors:10UF-16V-0603
- added C104, C105: 1uF 16V, ds_capacitors:1UF-16V0201
- added C125, C126, C93, C94, C99: 4.7uF 25V, ds_capacitors:4.7UF-25V0402
- added C127, C128: 12pF 50V, ds_capacitors:12PF-50V0201
- added C132, C135: 10uF 50V, ds_capacitors:10UF-50V-0805
- added C86: 27pF 50V, ds_capacitors:27PF-50V0201
- added DBGY, UARY: Yellow, ds_LED:LED-YELLOWLED-0603
- added G2R, PORT2, PORT4: Red, ds_LED:LED-REDLED-0603
- added IC10, IC7: SN74LVC541ARGYR, ds_ic_logic:74LVC541A
- added IC11: FT4232HL, ds_ic_peripherals:FT4232HL
- added IC12: 93LC56BT-I/OT, ds_ic_memory:93LC56BT-I/OT
- added IC13, IC25: MIC5504-3.3YM5, ds_ic_vreg:MIC5504-3.3YM5-TR
- added IC14: LMV611MFX/NOPB, ds_ic_opa:LMV611MFX
- added IC15, IC16, IC17: TXS0108ERGYR, ds_ic_peripherals:TXB0108RGY
- added IC18, IC19, IC20: TLV3501AIDBVR, ds_ic_opa:TLV3501AIDB
- added IC21: RP2040, ds_ic_mcu:RP2040
- added IC22: (no value), ds_ic_memory:W25Q128JVP
- added IC23, IC24: 74AUP1T17GWH, ds_ic_logic:74AUP1T17GW
- added IC8: CAT24C256HU4IGT3, ds_ic_memory:CAT24C256-HU4
- added IC9: CY7C68013A-56LTXC, ds_ic_mcu:CY7C68013A-56QFNLFXC
- added J7: JUMPER-NO, ds_passive:JUMPER-NO
- added JTAG: 62701021721, Wurth_Connectors_WR-BHD:6270XX21721_62701021721
- added LA: 62702021721, Wurth_Connectors_WR-BHD:6270XX21721_62702021721
- added R35, R38, R39: 10K 1%, ds_resistor:10K-1%0402
- added R36, R45, R47, R65: 10K 1%, ds_resistor:10K-1%0201
- added R37, R41, R42: 100K 1%, ds_resistor:100K-1%0201
- added R40: 15K 1%, ds_resistor:15K-1%0201
- added R43, R44, R48: 1K 1%, ds_resistor:1K-1%0603
- added R46: 7.87K 1%, ds_resistor:7.87K-1%0201
- added R49: 4.3K 1%, ds_resistor:4.3K-1%0201
- added R50, R53: 1K 1%, ds_resistor:1K-1%0201
- added R51, R52: 27R 1%, ds_resistor:27R-1%0201
- added R54, R55, R56, R57, R58: 1K 1%, ds_resistor:1K-1%0402
- added R59, R60, R61, R62, R63, R64: 100R 1%, ds_resistor:100R-1%0201
- added RN1, RN10, RN2, RN3, RN4, RN7, RN8, RN9: 100R 1%, ds_resistor:100R-1%_ARRAY0603X4-1206
- added RN11, RN12, RN5, RN6: 100K 1%, ds_resistor:100K-1%_ARRAY0603X4-1206
- added RPDBUG, RPUART: SM03B-SRSS-TB, ds_con:SM03B-SRSS-TB
- added SW1, SW2: B3U-1000P, ds_passive:B3U-1000P
- added T1, T2: (no value), ds_active:BSS138
- added UART1, UART2: 62731020621, Wurth_Connectors_WR-BHD:6273XX20621_62731020621
- added X1: 24MHz, Wurth_Quartz Crystals & Oscillators_WE-XTAL:WE-XTAL_CFPX-180_830108207709
- added X2: 24MHz, Wurth_Quartz Crystals & Oscillators_WE-XTAL:WE-XTAL_CFPX-180_830058149
- added X3, X4: 12MHz, Wurth_Quartz Crystals & Oscillators_WE-XTAL:WE-XTAL_CFPX-180_830055295
- C1, C13, C2, C3, C4, C5: value 100nF 16V -> 100nF 25V; device ds_capacitors:100NF-16V-0201 -> ds_capacitors:100NF-25V-0402
- C10: value 100nF 16V -> 1nF; device ds_capacitors:100NF-16V-0201 -> ds_passive:C-0402
- C11, C12, C6, C80, C9: value 100nF 16V -> 10uF 50V; device ds_capacitors:100NF-16V-0201 -> ds_capacitors:10UF-50V-0805
- C14, C15, C16: value 10nF 16V -> 100nF 25V; device ds_capacitors:10NF-16V-0201 -> ds_capacitors:100NF-25V-0402
- C21: value 22uF 16V -> 10nF 16V; device ds_capacitors:22UF-16V-0805 -> ds_capacitors:10NF-16V-0201
- C23: value 10nF 16V -> 100nF 16V; device ds_capacitors:10NF-16V-0201 -> ds_capacitors:100NF-16V-0201
- C26, C28, C30, C32, C34, C35, C36, C39: value 100nF 16V -> 10nF 16V; device ds_capacitors:100NF-16V-0201 -> ds_capacitors:10NF-16V-0201
- C29: value 22uF 16V -> 100nF 16V; device ds_capacitors:22UF-16V-0805 -> ds_capacitors:100NF-16V-0201
- C37, C38: value 10uF 50V -> 10nF 16V; device ds_capacitors:10UF-50V-0805 -> ds_capacitors:10NF-16V-0201
- C42, C65: value 100nF 16V -> 1uF 16V; device ds_capacitors:100NF-16V-0201 -> ds_capacitors:1UF-16V0201
- C43: value 100nF 16V -> 8pF 50V; device ds_capacitors:100NF-16V-0201 -> ds_capacitors:8PF-50V0201
- C44: value 10uF 50V -> 8pF 50V; device ds_capacitors:10UF-50V-0805 -> ds_capacitors:8PF-50V0201
- C45: value 10uF 50V -> 22uF 25V; device ds_capacitors:10UF-50V-0805 -> ds_capacitors:22UF-25V-0805
- C46: value 100nF 25V -> 10uF 16V; device ds_capacitors:100NF-25V-0402 -> ds_capacitors:10UF-16V-0805
- C47: value 100nF 25V -> 10nF 50V; device ds_capacitors:100NF-25V-0402 -> ds_capacitors:10NF-50V-0805
- C48: value 100nF 25V -> 10nF 16V; device ds_capacitors:100NF-25V-0402 -> ds_capacitors:10NF-16V-0201
- C49: value 100nF 25V -> DNI; device ds_capacitors:100NF-25V-0402 -> ds_capacitors:C-0201
- C50: value 1nF -> 10nF 25V; device ds_passive:C-0402 -> ds_capacitors:10NF-25V-0402
- C51: value 18pF 25V -> 10nF 50V; device ds_capacitors:18PF-25V-0201 -> ds_capacitors:10NF-50V-0805
- C52: value 18pF 25V -> 330uF 25V; device ds_capacitors:18PF-25V-0201 -> ds_capacitors:330UF-25V6.3X7.7(DXL)
- C53: value 100nF 16V -> 22uF 16V; device ds_capacitors:100NF-16V-0201 -> ds_capacitors:22UF-16V-0805
- C56, C58, C61: value 150uF 35V -> 100nF 16V; device ds_capacitors:150UF-35V-6.3X5.5 -> ds_capacitors:100NF-16V-0201
- C59, C60, C64: value 100nF 16V -> 150uF 35V; device ds_capacitors:100NF-16V-0201 -> ds_capacitors:150UF-35V-6.3X5.5
- C66, C74: value 100nF 16V -> 100nF 25V; device ds_capacitors:100NF-16V-0603 -> ds_capacitors:100NF-25V-0201
- C67: value 1nF 16V -> 100nF 25V; device ds_capacitors:1NF-16V-0402 -> ds_capacitors:100NF-25V-0201
- C68, C69, C72, C73, C77: value 100nF 16V -> 100nF 25V; device ds_capacitors:100NF-16V-0201 -> ds_capacitors:100NF-25V-0201
- C70: value 10nF 16V -> 100nF 25V; device ds_capacitors:10NF-16V-0201 -> ds_capacitors:100NF-25V-0201
- C71: value DNI -> 100nF 25V; device ds_capacitors:C-0201 -> ds_capacitors:100NF-25V-0201
- C75: value 1nF 16V -> 12pF 50V; device ds_capacitors:1NF-16V-0402 -> ds_capacitors:12PF-50V0201
- C76: value 100nF 16V -> 12pF 50V; device ds_capacitors:100NF-16V-0201 -> ds_capacitors:12PF-50V0201
- C78: value 10uF 16V -> 100nF 25V; device ds_capacitors:10UF-16V-0805 -> ds_capacitors:100NF-25V-0201
- C79: value 22uF 16V -> 100nF 25V; device ds_capacitors:22UF-16V-0805 -> ds_capacitors:100NF-25V-0201
- C81: value 10nF 50V -> 10uF 50V; device ds_capacitors:10NF-50V-0805 -> ds_capacitors:10UF-50V-0805
- C82: value 22uF 25V -> 100nF 25V; device ds_capacitors:22UF-25V-0805 -> ds_capacitors:100NF-25V-0201
- C83: value 10nF 25V -> 100nF 25V; device ds_capacitors:10NF-25V-0402 -> ds_capacitors:100NF-25V-0201
- C84: value 10nF 50V -> 100nF 25V; device ds_capacitors:10NF-50V-0805 -> ds_capacitors:100NF-25V-0402
- C85: value 330uF 25V -> 27pF 50V; device ds_capacitors:330UF-25V6.3X7.7(DXL) -> ds_capacitors:27PF-50V0201
- D1: value Red -> 1SS294; device ds_LED:LED-REDLED-0603 -> diode:BAT54
- D10: value (none) -> Red; device ds_ic_peripherals:TPD4EUSB30 -> ds_LED:LED-REDLED-0603
- D8: value (none) -> 1N4148SOD-123; device ds_ic_peripherals:TPD4EUSB30 -> adafruit:DIODE_SOD-123FL
- D9: value (none) -> MBRS540T3G; device ds_ic_peripherals:TPD4EUSB30 -> diode:DIODE-SMC
- IC1: value TUSB7340RKMR -> UPD720201K8-701-BAC-A; device ds_ic_peripherals:TUSB7340RKMR -> ds_ic_peripherals:UPD720201
- IC2: value 24LC01BT-I/OT -> TPS5450DDAR; device 52101-101-REV-A_v16:MEMORY-ATMEL_AT24CS01-ST -> ds_ic_vreg:TPS5450
- IC3: value TPS2560DRCR -> TPS74401RGWT; device ds_ic_vreg:TPS2560DRCR -> ds_ic_vreg:TPS74401RGWT
- IC5: value TPS74401RGWT -> TPS2560DRCR; device ds_ic_vreg:TPS74401RGWT -> ds_ic_vreg:TPS2560DRCR
- IC6: value TPS5450DDAR -> MIC5504-3.3YM5-TR; device ds_ic_vreg:TPS5450 -> MCU:MIC5504-3.3YM5-TR
- J3: value JUMPER-NO -> JUMPER-3; device ds_passive:JUMPER-NO -> ds_passive:JUMPER-3
- J4: value 692141030100 -> 66100511622; device Wurth_Connectors_WR-USB:692141030100 -> Wurth_Connectors_WR-WTB:66100511622
- R1: value 10K 1% -> 0R 1%; device ds_resistor:10K-1%0201 -> ds_resistor:0R0201
- R10: value DNI -> 1.37K 1%; device ds_resistor:R-0201 -> ds_resistor:1.37K-1%0201
- R11: value DNI -> 4.42K 1%; device ds_resistor:R-0201 -> ds_resistor:4.42K-1%0201
- R12: value DNI -> 1K 1%; device ds_resistor:R-0201 -> ds_resistor:1K-1%0402
- R13, R14: value 0R 1% -> 30.9K 1%; device ds_resistor:0R0201 -> ds_resistor:30.9K-1%0201
- R15, R16, R5: value 10K 1% -> 1K 1%; device ds_resistor:10K-1%0201 -> ds_resistor:1K-1%0402
- R17, R22: value 30.9K 1% -> 1K 1%; device ds_resistor:30.9K-1%0201 -> ds_resistor:1K-1%0402
- R19: value 1K 1% -> 100K 1%; device ds_resistor:1K-1%0402 -> ds_resistor:100K-1%0201
- R2: value DNI -> BLM21PG600SN1; device ds_resistor:R-0201 -> ds_passive:R0603
- R20, R21: value 10K 1% -> 3.3K 1%; device ds_resistor:10K-1%0201 -> ds_resistor:3.3K-1%0201
- R23: value 1K 1% -> 2K 1%; device ds_resistor:1K-1%0402 -> ds_resistor:2K-1%0201
- R24, R28: value 1K 1% -> 10K 1%; device ds_resistor:1K-1%0402 -> ds_resistor:10K-1%0201
- R25: value 1M 1% -> 10K 1%; device ds_resistor:1M-1%0402 -> ds_resistor:10K-1%0201
- R26: value 4.7K 1% -> 10K 1%; device ds_resistor:4.7K-1%0201 -> ds_resistor:10K-1%0201
- R27: value 1M 1% -> 4.7K 1%; device ds_resistor:1M-1%0402 -> ds_resistor:4.7K-1%0201
- R29: value 10K 1% -> 12K 1%; device ds_resistor:10K-1%0201 -> ds_resistor:12K-1%0201
- R3: value 0R 1% -> 10K 1%; device ds_resistor:0R0201 -> ds_resistor:10K-1%0201
- R30: value 1.87K 1% -> 1K 1%; device ds_resistor:1.87K-1%0201 -> ds_resistor:1K-1%0201
- R31: value 4.99K 1% -> 4.7K 1%; device ds_resistor:4.99K-1%0201 -> ds_resistor:4.7K-1%0201
- R32: value 10K 1% -> 4.7K 1%; device ds_resistor:10K-1%0402 -> ds_resistor:4.7K-1%0201
- R33: value 3.16K 1% -> 10K 1%; device ds_resistor:3.16K-1%0402 -> ds_resistor:10K-1%0402
- R34: value 1K 1% -> 22K 1%; device ds_resistor:1K-1%0402 -> ds_resistor:22K-1%0402
- R4: value 4.7K 1% -> 1.6K 1%; device ds_resistor:4.7K-1%0201 -> ds_resistor:1.6K-1%0201
- R6: value 9.09K 1% -> 4.7K 1%; device ds_resistor:9.09K-1%0201 -> ds_resistor:4.7K-1%0201
- R7: value DNI -> 10K 1%; device ds_resistor:R-0201 -> ds_resistor:10K-1%0402
- R8: value DNI -> 3.16K 1%; device ds_resistor:R-0201 -> ds_resistor:3.16K-1%0402
- R9: value DNI -> 10K 1%; device ds_resistor:R-0201 -> ds_resistor:10K-1%0201
- renumbered D13 to PGOOD5, D2 to PORT1, D4 to PORT3
Connections:
- removed net LED_1V1: D11.C, R28.1
- removed net N$37: IC1A.FREQSEL, R4.1
- removed net N$54: IC1A.GPIO[0], R10.2
- removed net N$55: IC1A.GPIO[1], R9.2
- removed net N$56: IC1A.GPIO[2], R8.2
- removed net N$57: IC1A.GPIO[3], R7.2
- removed net N$59: IC1A.R1EXT, R6.1
- removed net PCIE_CAPTX_N: C36.2, PCIE-1X1.PER_N0
- removed net PCIE_CAPTX_P: C35.2, PCIE-1X1.PER_P0
- removed net SHIELD-1: C66.1, C67.1, J4USBA.SHIELD, J5USBA.SHIELD, R25.1
- removed net SHIELD-2: C74.1, C75.1, J4USBB.SHIELD, J5USBB.SHIELD, R27.1
- removed net USB1_CSSTX_N: C64.1, J4USBA.STDA_SSTX-
- removed net USB1_CSSTX_P: C65.1, J4USBA.STDA_SSTX+
- removed net USB2_CSSTX_N: C68.1, J5USBA.STDA_SSTX-
- removed net USB2_CSSTX_P: C69.1, J5USBA.STDA_SSTX+
- removed net USB3_CSSTX_N: C72.1, J4USBB.STDA_SSTX-
- removed net USB3_CSSTX_P: C73.1, J4USBB.STDA_SSTX+
- removed net USB4_CSSTX_N: C76.1, J5USBB.STDA_SSTX-
- removed net USB4_CSSTX_P: C77.1, J5USBB.STDA_SSTX+
- new net !CTS1: IC11.CDBUS3, IC16.B5
- new net !CTS1_OUT: IC16.A5, UART1.5
- new net !CTS2: IC11.DDBUS3, IC17.B5
- new net !CTS2_OUT: IC17.A5, UART2.6
- new net !DCD1: IC11.CDBUS6, IC16.B2
- new net !DCD1_OUT: IC16.A2, UART1.10
- new net !DCD2: IC11.DDBUS6, IC17.B2
- new net !DCD2_OUT: IC17.A2, UART2.1
- new net !DSR1: IC11.CDBUS5, IC16.B3
- new net !DSR1_OUT: IC16.A3, UART1.9
- new net !DSR2: IC11.DDBUS5, IC17.B3
- new net !DSR2_OUT: IC17.A3, UART2.2
- new net !DTR1: IC11.CDBUS4, IC16.B4
- new net !DTR1_OUT: IC16.A4, UART1.4
- new net !DTR2: IC11.DDBUS4, IC17.B4
- new net !DTR2_OUT: IC17.A4, UART2.7
- new net !PECREQ: !REQ.TP, IC1G$1.PECREQB
- new net !RI1: IC11.CDBUS7, IC16.B1
- new net !RI1_OUT: IC16.A1, UART1.3
- new net !RI2: IC11.DDBUS7, IC17.B1
- new net !RI2_OUT: IC17.A1, UART2.8
- new net !RTS1: IC11.CDBUS2, IC16.B6
- new net !RTS1_OUT: IC16.A6, UART1.7
- new net !RTS2: IC11.DDBUS2, IC17.B6
- new net !RTS2_OUT: IC17.A6, UART2.4
- new net !SMI: !SMI.TP, IC1G$1.SMIB
- new net !SPI_CS: IC1G$1.SPICSB
- new net +1V05: C17.1, C18.1, C19.1, C20.1, C21.1, C22.1, C23.1, C24.1, C25.1, C26.1, C27.1, C28.1, C29.1, C53.1, IC1G$2.VDD10@1, IC1G$2.VDD10@2, IC1G$2.VDD10@3, IC1G$2.VDD10@4, IC1G$2.VDD10@5, IC1G$2.VDD10@6, IC1G$2.VDD10@7, IC1G$2.VDD10@8, IC1G$2.VDD10@9, IC3.OUT@1, IC3.OUT@2, IC3.OUT@3, IC3.OUT@4, R10.1
- new net +1V8: C95.1, C96.1, C97.1, C98.1, C99.1, IC11.VCORE@1, IC11.VCORE@2, IC11.VCORE@3, IC11.VREGOUT
- new net +3V3B: C66.1, C67.1, C68.1, C69.1, C70.1, C71.1, C72.1, C73.1, C74.1, C77.1, C78.1, C81.1, C82.1, C83.1, D8.C, IC10.VCC, IC6.VOUT, IC7.VCC, IC8.VCC, IC9.AVCC, IC9.VCC, IC9.WAKEUP, R19.1, R20.2, R21.2, RN11A.2, RN11B.2, RN11C.2, RN11D.2, RN12A.2, RN12B.2, RN12C.2, RN12D.2, RN5A.2, RN5B.2, RN5C.2, RN5D.2, RN6A.2, RN6B.2, RN6C.2, RN6D.2
- new net +3V3C: C102.1, C103.1, C109.1, C111.1, C113.1, C84.1, C87.1, C88.1, C89.1, C90.1, C91.1, C92.1, C93.1, C94.1, IC11.VCCIO@1, IC11.VCCIO@2, IC11.VCCIO@3, IC11.VCCIO@4, IC11.VPHY, IC11.VPLL, IC11.VREGIN, IC12.VCC, IC13.VOUT, IC15.VCCB, IC16.VCCB, IC17.VCCB, R24.1, R25.1, R26.1, R31.1, R32.1, R33.1
- new net +3V3D: C117.1, C118.1, C119.1, C120.1, C121.1, C122.1, C125.1, C129.1, C130.1, C131.1, C134.1, C135.1, IC21.ADC_AVDD, IC21.IOVDD, IC21.USB_VDD, IC21.VREG_VIN, IC22.VCC, IC23.VCC, IC24.VCC, IC25.VOUT, R65.1
- new net 4232R_RESET: R27.2, R28.1, R30.1
- new net 4232_RESET: IC11.!RESET, R30.2
- new net BOOT: R53.1, SW2.P$1
- new net BUF_PB0: IC7.Y0, RN3A.1
- new net BUF_PB1: IC7.Y1, RN3B.1
- new net BUF_PB2: IC7.Y2, RN3C.1
- new net BUF_PB3: IC7.Y3, RN3D.1
- new net BUF_PB4: IC7.Y4, RN4A.1
- new net BUF_PB5: IC7.Y5, RN4B.1
- new net BUF_PB6: IC7.Y6, RN4C.1
- new net BUF_PB7: IC7.Y7, RN4D.1
- new net BUF_PD0: IC10.Y0, RN9A.1
- new net BUF_PD1: IC10.Y1, RN9B.1
- new net BUF_PD2: IC10.Y2, RN9C.1
- new net BUF_PD3: IC10.Y3, RN9D.1
- new net BUF_PD4: IC10.Y4, RN10A.1
- new net BUF_PD5: IC10.Y5, RN10B.1
- new net BUF_PD6: IC10.Y6, RN10C.1
- new net BUF_PD7: IC10.Y7, RN10D.1
- new net CH0: LA.17, RN1A.1
- new net CH1: LA.15, RN1B.1
- new net CH10: LA.8, RN7C.1
- new net CH11: LA.10, RN7D.1
- new net CH12: LA.12, RN8A.1
- new net CH13: LA.14, RN8B.1
- new net CH14: LA.16, RN8C.1
- new net CH15: LA.18, RN8D.1
- new net CH2: LA.13, RN1C.1
- new net CH3: LA.11, RN1D.1
- new net CH4: LA.9, RN2A.1
- new net CH5: LA.7, RN2B.1
- new net CH6: LA.5, RN2C.1
- new net CH7: LA.3, RN2D.1
- new net CH8: LA.4, RN7A.1
- new net CH9: LA.6, RN7B.1
- new net CHI0: IC7.A0, RN1A.2, RN5A.1
- new net CHI1: IC7.A1, RN1B.2, RN5B.1
- new net CHI10: IC10.A2, RN11C.1, RN7C.2
- new net CHI11: IC10.A3, RN11D.1, RN7D.2
- new net CHI12: IC10.A4, RN12A.1, RN8A.2
- new net CHI13: IC10.A5, RN12B.1, RN8B.2
- new net CHI14: IC10.A6, RN12C.1, RN8C.2
- new net CHI15: IC10.A7, RN12D.1, RN8D.2
- new net CHI2: IC7.A2, RN1C.2, RN5C.1
- new net CHI3: IC7.A3, RN1D.2, RN5D.1
- new net CHI4: IC7.A4, RN2A.2, RN6A.1
- new net CHI5: IC7.A5, RN2B.2, RN6B.1
- new net CHI6: IC7.A6, RN2C.2, RN6C.1
- new net CHI7: IC7.A7, RN2D.2, RN6D.1
- new net CHI8: IC10.A0, RN11A.1, RN7A.2
- new net CHI9: IC10.A1, RN11B.1, RN7B.2
- new net CLK: R62.2, RPDBUG.1
- new net COMP18_O: IC20.OUT, R48.1
- new net COMP25_O: IC19.OUT, R44.1
- new net COMP33_O: IC18.OUT, R43.1
- new net D25: R35.2, T2.D
- new net D33: R34.2, T1.D
- new net DIO: R63.2, R64.2, RPDBUG.3
- new net EECLK: IC11.EECLK, IC12.CLK, R26.2
- new net EECS: IC11.EECS, IC12.!CS, R24.2
- new net EEDATA: IC11.EEDATA, IC12.DI, R23.2, R25.2
- new net FT_SCL: IC11.ADBUS0, IC15.B8, R32.2
- new net FT_SCL_OUT: IC15.A8
- new net FT_SDA: IC11.ADBUS1, IC11.ADBUS2, IC15.B7, R31.2
- new net FT_SDA_OUT: IC15.A7
- new net GPIO12: IC21.GPIO12, R62.1
- new net GPIO13: IC21.GPIO13, IC24.Y
- new net GPIO14: IC21.GPIO14, R63.1
- new net GPIO15: IC21.GPIO15, R57.1
- new net GPIO16: IC21.GPIO16, R58.1
- new net GPIO2: IC21.GPIO2, R54.1
- new net GPIO4: IC21.GPIO4, R59.1
- new net GPIO5: IC21.GPIO5, IC23.Y
- new net GPIO6: IC21.GPIO6, R60.1
- new net GPIO7: IC21.GPIO7, R55.1
- new net GPIO8: IC21.GPIO8, R56.1
- new net ILIM12: IC4.ILIM, R13.1
- new net ILIM34: IC5.ILIM, R14.1
- new net JTAG_TDO: J1.P$2, PCIE-1X1.JTAG_TDO
- new net KEY: JTAG.7
- new net LA_LED: D10.C, R22.1
- new net LED_3V: PGOOD3.A, R5.2
- new net LED_5V: PGOOD5.A, R12.2
- new net N$11: C128.1, R50.2, X4.2
- new net N$12: 2V5.A, R44.2
- new net N$13: IC21.XOUT, R50.1
- new net N$14: 1V8.A, R48.2
- new net N$15: J7.P$2, JTAG.1
- new net N$16: G2R.A, R54.2
- new net N$17: DBGG.A, R57.2
- new net N$18: DBGY.A, R58.2
- new net N$19: R56.2, UARY.A
- new net N$20: R55.2, UARG.A
- new net N$21: IC24.A, R64.1
- new net N$24: IC23.A, R61.1
- new net N$8: 3V3.A, R43.2
- new net PA0: IC9.PA0
- new net PA1: D10.A, IC9.PA1
- new net PA2: IC9.PA2
- new net PA3: IC9.PA3
- new net PA4: IC9.PA4
- new net PA5: IC9.PA5
- new net PA6: IC9.PA6
- new net PA7: IC9.PA7
- new net PB0: IC9.PB0, RN3A.2
- new net PB1: IC9.PB1, RN3B.2
- new net PB2: IC9.PB2, RN3C.2
- new net PB3: IC9.PB3, RN3D.2
- new net PB4: IC9.PB4, RN4A.2
- new net PB5: IC9.PB5, RN4B.2
- new net PB6: IC9.PB6, RN4C.2
- new net PB7: IC9.PB7, RN4D.2
- new net PCIE_CTX_N: C8.2, PCIE-1X1.PER_N0
- new net PCIE_CTX_P: C7.2, PCIE-1X1.PER_P0
- new net PD0: IC9.PD0, RN9A.2
- new net PD1: IC9.PD1, RN9B.2
- new net PD2: IC9.PD2, RN9C.2
- new net PD3: IC9.PD3, RN9D.2
- new net PD4: IC9.PD4, RN10A.2
- new net PD5: IC9.PD5, RN10B.2
- new net PD6: IC9.PD6, RN10C.2
- new net PD7: IC9.PD7, RN10D.2
- new net PH: C50.2, D9.C, IC2.PH, L1.2
- new net QSPI_SCLK: IC21.QSPI_SCLK, IC22.CLK
- new net QSPI_SD0: IC21.QSPI_SD0, IC22.DI/IO0
- new net QSPI_SD1: IC21.QSPI_SD1, IC22.DO/IO1
- new net QSPI_SD2: IC21.QSPI_SD2, IC22.!WP!/IO2
- new net QSPI_SD3: IC21.QSPI_SD3, IC22.!HOLD!/IO3
- new net QSPI_SS: IC21.QSPI_SS_N, IC22.!CS, R53.2
- new net RESET: C65.1, D8.A, IC9.!RESET, R19.2
- new net RUN: IC21.RUN, R65.2, SW1.P$1
- new net RXD1: IC11.CDBUS1, IC16.B7
- new net RXD1_OUT: IC16.A7, UART1.8
- new net RXD2: IC11.DDBUS1, IC17.B7
- new net RXD2_OUT: IC17.A7, UART2.3
- new net SPI_MISO: IC1G$1.SPISI
- new net SPI_MOSI: IC1G$1.SPISO
- new net SPI_SCK: IC1G$1.SPISCK
- new net SWCLK: IC21.SWCLK
- new net SWDIO: IC21.SWDIO
- new net TCK/SCK: IC11.BDBUS0, IC15.B4
- new net TCK/SCK_OUT: IC15.A4, JTAG.4
- new net TDI/DO: IC11.BDBUS1, IC15.B3
- new net TDI/DO_OUT: IC15.A3, JTAG.8
- new net TDO/DI: IC11.BDBUS2, IC15.B2
- new net TDO/DI_OUT: IC15.A2, JTAG.6
- new net TMS/CS: IC11.BDBUS3, IC15.B1
- new net TMS/CS_OUT: IC15.A1, JTAG.2
- new net TRESET: IC11.BDBUS4
- new net TRESET_OUT: JTAG.10
- new net TXD1: IC11.CDBUS0, IC16.B8
- new net TXD1_OUT: IC16.A8, UART1.6
- new net TXD2: IC11.DDBUS0, IC17.B8
- new net TXD2_OUT: IC17.A8, UART2.5
- new net UART1_RX: R60.2, R61.2, RPUART.3
- new net UART1_TX: R59.2, RPUART.1
- new net USB_PID_N: IC21.USB_DM, R51.2
- new net USB_PID_P: IC21.USB_DP, R52.1
- new net VDIV_BUF: C104.1, IC14.+IN, R33.2, R34.1, R35.1
- new net VREF_LOGIC: C107.1, C108.1, C110.1, C112.1, IC14.-IN, IC14.OUT, IC15.OE, IC15.VCCA, IC16.OE, IC16.VCCA, IC17.OE, IC17.VCCA, IC18.+IN, IC19.+IN, IC20.+IN, J7.P$1, R37.1, R41.1, R42.1
- new net VSEL_1V8: IC11.ADBUS6, R39.1, T2.G
- new net VSEL_2V5: IC11.ADBUS7, R38.1, T1.G
- new net V_COMP18: IC20.-IN, R47.2, R49.1
- new net V_COMP25: IC19.-IN, R45.2, R46.1
- new net V_COMP33: IC18.-IN, R36.2, R40.1
- new net XIN: C75.1, IC9.XTALIN, X2.1
- new net XOUT: C76.1, IC9.XTALOUT, X2.2
- net !GRST: now also !RST.TP, C42.1, C54.1, D1.A, IC1G$1.PONRSTB, IC3.PG, R3.2, R9.2; no longer C80.1, IC1A.!GRST, IC5.PG, R29.2
- net !OVERCUR1: now also IC1G$1.OCI1B, IC4.!FAULT1; no longer IC1A.!OVERCUR1, IC3.!FAULT2
- net !OVERCUR2: now also IC1G$1.OCI2B, IC4.!FAULT2; no longer IC1A.!OVERCUR2, IC4.!FAULT1
- net !OVERCUR3: now also IC1G$1.OCI3B, IC5.!FAULT1; no longer IC1A.!OVERCUR3, IC3.!FAULT1
- net !OVERCUR4: now also IC1G$1.OCI4B, IC5.!FAULT2; no longer IC1A.!OVERCUR4, IC4.!FAULT2
- net !PERST: now also !PERST.TP, IC1G$1.PERSTB; no longer IC1A.!PERST
- net !PWRON1: now also IC1G$1.PPON1, IC4.EN1; no longer IC1A.!PWRON1, IC3.EN2
- net !PWRON2: now also IC1G$1.PPON2, IC4.EN2; no longer IC1A.!PWRON2, IC4.EN1
- net !PWRON3: now also IC1G$1.PPON3, IC5.EN1; no longer IC1A.!PWRON3, IC3.EN1
- net !PWRON4: now also IC1G$1.PPON4, IC5.EN2; no longer IC1A.!PWRON4, IC4.EN2
- net !WAKE: now also C10.1, IC1G$1.PEWAKEB, R1.2; no longer C50.1, IC1A.!WAKE, R3.2
- net !WAKE_R: now also R1.1; no longer R3.1
- net +12V: now also C1.1, C2.1, C3.1, C4.1, C45.1, C47.1, C5.1, C6.1, C9.1, IC2.VIN; no longer C37.1, C38.1, C39.1, C40.1, C41.1, C42.1, C43.1, C81.1, C82.1, IC6.VIN
- net +1V1: now also C123.1, C124.1, C126.1, IC21.DVDD, IC21.VREG_VOUT; no longer C1.1, C10.1, C11.1, C12.1, C13.1, C14.1, C15.1, C16.1, C17.1, C18.1, C19.1, C2.1, C20.1, C21.1, C3.1, C4.1, C5.1, C6.1, C7.1, C79.1, C8.1, C9.1, IC1B.VDD11@1, IC1B.VDD11@10, IC1B.VDD11@11, IC1B.VDD11@12, IC1B.VDD11@13, IC1B.VDD11@14, IC1B.VDD11@15, IC1B.VDD11@16, IC1B.VDD11@17, IC1B.VDD11@18, IC1B.VDD11@19, IC1B.VDD11@2, IC1B.VDD11@3, IC1B.VDD11@4, IC1B.VDD11@5, IC1B.VDD11@6, IC1B.VDD11@7, IC1B.VDD11@8, IC1B.VDD11@9, IC5.OUT@1, IC5.OUT@2, IC5.OUT@3, IC5.OUT@4, R30.1
- net +3V3: now also C36.1, C38.1, C39.1, C40.1, C41.1, C46.1, D1.C, IC1G$2.VDD33@1, IC1G$2.VDD33@2, IC1G$2.VDD33@3, IC1G$2.VDD33@4, IC1G$2.VDD33@5, IC1G$2.VDD33@6, IC3.BIAS, IC3.IN@1, IC3.IN@2, IC3.IN@3, IC3.IN@4, R2.1, R3.1, R5.1, R6.1; no longer C31.1, C33.1, C53.1, C78.1, D11.A, FB1.1, IC1B.VDD33@1, IC1B.VDD33@2, IC1B.VDD33@3, IC1B.VDD33@4, IC1B.VDD33@5, IC2.VCC, IC5.BIAS, IC5.IN@1, IC5.IN@2, IC5.IN@3, IC5.IN@4, R1.1, R10.1, R11.1, R12.1, R15.1, R16.1, R20.1, R21.1, R26.1, R29.1, R7.1, R8.1
- net +3V3A: now also C31.1, C33.1, C35.1, C37.1, IC1G$2.AVDD33@1, IC1G$2.AVDD33@2, R2.2; no longer C22.1, C23.1, C24.1, C25.1, C26.1, C27.1, C28.1, C29.1, FB1.2, IC1B.VDDA_3P3@1, IC1B.VDDA_3P3@2, IC1B.VDDA_3P3@3, IC1B.VDDA_3P3@4, IC1B.VDDA_3P3@5, IC1B.VDDA_3P3@6, IC1B.VDDA_3P3@7, IC1B.VDDA_3P3@8
- net +3V3_AUX: now also AUX3.TP
- net +5V: now also C51.1, C52.+, C55.1, C56.1, IC5.IN@1, IC5.IN@2, R12.1, R7.1; no longer C54.1, C59.1, C84.1, C85.+, IC3.IN@1, IC3.IN@2, R32.1, R34.1
- net BOOT_5V: now also C50.1, IC2.BOOT; no longer C83.1, IC6.BOOT
- net DS1_VBUS: now also C59.+, C79.1, C80.1, IC4.OUT1, IC6.EN, IC6.VIN, R17.1; no longer C58.+, IC3.OUT2, J4USBA.VBUS, R16.2, R18.1
- net DS2_VBUS: now also C100.1, C101.1, C105.1, C106.1, C114.1, C115.1, C116.1, C61.1, C63.+, IC13.EN, IC13.VIN, IC14.V+, IC18.V+, IC19.V+, IC20.V+, IC4.OUT2, R15.1, R27.1, R36.1, R45.1, R47.1; no longer C60.1, C61.+, IC4.OUT1, J5USBA.VBUS, R20.2, R24.1
- net DS3_VBUS: now also C132.1, C133.1, C58.1, C60.+, IC25.EN, IC25.VIN, IC5.OUT1, R18.1; no longer C55.1, C56.+, IC3.OUT1, J4USBB.VBUS, R15.2, R19.1
- net DS4_VBUS: now also C64.+, IC5.OUT2, J4.1, R16.1; no longer C63.+, IC4.OUT2, J5USBB.VBUS, R21.2, R23.1
- net EN_1V1: now also C48.1, IC3.EN, R6.2; no longer C70.1, IC5.EN, R26.2
- net FB_1V1: now also IC3.FB, R10.2, R11.1; no longer IC5.FB, R30.2, R31.1
- net FB_5V: now also IC2.VSENSE, R7.2, R8.1; no longer IC6.VSENSE, R32.2, R33.1
- net GND: now also 1V8.C, 2V5.C, 3V3.C, C100.2, C101.2, C102.2, C103.2, C104.2, C105.2, C106.2, C107.2, C108.2, C109.2, C110.2, C111.2, C112.2, C113.2, C114.2, C115.2, C116.2, C117.2, C118.2, C119.2, C120.2, C121.2, C122.2, C123.2, C124.2, C125.2, C126.2, C127.2, C128.2, C129.2, C130.2, C131.2, C132.2, C133.2, C134.2, C135.2, C35.2, C36.2, C52.-, C56.2, C58.2, C59.-, C60.-, C61.2, C64.-, C65.2, C68.2, C69.2, C72.2, C73.2, C76.2, C77.2, C83.2, C85.2, C86.2, C87.2, C88.2, C89.2, C90.2, C91.2, C92.2, C93.2, C94.2, C95.2, C96.2, C97.2, C98.2, C99.2, D9.A, DBGG.C, DBGY.C, G2R.C, IC10.!OE1, IC10.!OE2, IC10.GND, IC11.AGND, IC11.GND@1, IC11.GND@2, IC11.GND@3, IC11.GND@4, IC11.GND@5, IC11.GND@6, IC11.GND@7, IC11.GND@8, IC11.TEST, IC12.GND, IC13.GND, IC14.V-, IC15.GND, IC16.GND, IC17.GND, IC18.SHDN, IC18.V-, IC19.SHDN, IC19.V-, IC1G$1.IC(L), IC1G$2.GND, IC2.POWERPAD, IC20.SHDN, IC20.V-, IC21.GND, IC21.TESTEN, IC22.GND, IC23.GND, IC24.GND, IC25.GND, IC3.THERMAL_PAD, IC5.PAD, IC7.!OE1, IC7.!OE2, IC7.GND, IC8.A0, IC8.A1, IC8.A2, IC8.GND, IC8.WP, IC9.AGND, IC9.EPAD, IC9.GND, IC9.RESERVED, J3.2, J4.5, JTAG.3, JTAG.5, JTAG.9, LA.1, LA.19, LA.2, LA.20, PGOOD3.C, PORT2.C, PORT4.C, R11.2, R29.2, R37.2, R38.2, R39.2, R40.2, R41.2, R42.2, R46.2, R49.2, R8.2, RPDBUG.2, RPDBUG.SHLD, RPUART.2, RPUART.SHLD, SW1.P$2, SW2.P$2, T1.S, T2.S, UARG.C, UART1.2, UART2.9, UARY.C, X1.GND, X2.GND, X3.GND, X4.GND; no longer C50.2, C52.2, C56.-, C58.-, C59.2, C60.2, C61.-, C7.2, C8.2, C85.-, D1.C, D10.GND, D12.A, D3.C, D5.GND, D6.GND, D7.GND, D8.GND, D9.GND, IC1B.VSS@1, IC1B.VSS@2, IC1B.VSS_NC@1, IC1B.VSS_NC@2, IC1B.VSS_NC@3, IC1B.VSS_NC@4, IC1B.VSS_OSC, IC2.WP, IC3.PAD, IC5.THERMAL_PAD, IC6.POWERPAD, J1.P$2, J4USBA.GND, J4USBA.GND_DRAIN, J4USBB.GND, J4USBB.GND_DRAIN, J5USBA.GND, J5USBA.GND_DRAIN, J5USBB.GND, J5USBB.GND_DRAIN, R17.2, R2.2, R25.2, R27.2, R31.2, R33.2, R5.1, Y1.GND
- net JTAG_TDITDO: now also J1.P$1; no longer J3.P$1
- net LEDDS1: now also PORT2.A, R15.2; no longer D1.A, R18.2
- net LEDDS2: now also R18.2; no longer R24.2
- net LEDDS3: now also R17.2; no longer R19.2
- net LEDDS4: now also PORT4.A, R16.2; no longer D3.A, R23.2
- net N$1: now also IC21.GPIO0, J3.1; no longer IC1B.AUX_DET, J1.P$1, R1.2, R2.1
- net N$10: now also C86.1, IC11.OSCO, X3.2; no longer C83.2, D12.C, IC6.PH, L1.2
- net N$2: now also IC11.REF, R29.1; no longer J3.P$2, PCIE-1X1.JTAG_TDO
- net N$3: now also C85.1, IC11.OSCI, X3.1; no longer IC1A.!JTAG_RST, R5.2
- net N$4: now also C43.1, IC1G$1.XT1, X1.1; no longer C51.1, IC1A.XO, Y1.1
- net N$5: now also C44.1, IC1G$1.XT2, X1.2; no longer C52.1, IC1A.XI, Y1.2
- net N$6: now also IC12.DO, R23.1; no longer IC3.ILIM, R17.1
- net N$60: now also IC1G$1.RREF, R4.1; no longer IC1A.R1EXTRTN, R6.2
- net N$7: now also IC21.GPIO1, J3.3; no longer PGOOD5.A, R34.2
- net N$9: now also C127.1, IC21.XIN, X4.1; no longer IC4.ILIM, R22.1
- net PCIE_3V3: now also C11.1, C12.1, C13.1, C14.1, C15.1, C16.1; no longer C44.1, C45.1, C46.1, C47.1, C48.1, C49.1
- net PCIE_REFCLK_N: now also IC1G$1.PECLKP; no longer IC1A.PCIE_REFCLKN
- net PCIE_REFCLK_P: now also IC1G$1.PECLKN; no longer IC1A.PCIE_REFCLKP
- net PCIE_RX_N: now also IC1G$1.PERXN; no longer IC1A.PCIE_RXN
- net PCIE_RX_P: now also IC1G$1.PERXP; no longer IC1A.PCIE_RXP
- net PCIE_TX_N: now also C8.1, IC1G$1.PETXN; no longer C36.1, IC1A.PCIE_TXN
- net PCIE_TX_P: now also C7.1, IC1G$1.PETXP; no longer C35.1, IC1A.PCIE_TXP
- net SCL: now also IC8.SCL, IC9.SCL, R20.1; no longer IC1A.SCL, IC2.SCL, R11.2, R13.1
- net SDA: now also IC8.SDA, IC9.SDA, R21.1; no longer IC1A.SDA, IC2.SDA, R12.2, R14.1
- net SS: now also C49.1, IC3.SS; no longer C71.1, IC5.SS
- net USB1_DP_N: now also IC1G$1.U2DM1, IC9.DN; no longer D5.D1+, IC1A.USB_DM_DN1, J4USBA.D-
- net USB1_DP_P: now also IC1G$1.U2DP1, IC9.DP; no longer D5.D1-, IC1A.USB_DP_DN1, J4USBA.D+
- net USB1_SSRX_N: now also IC1G$1.U3RXDN1; no longer D5.D2+, IC1A.USB_SSRXN_DN1, J4USBA.STDA_SSRX-
- net USB1_SSRX_P: now also IC1G$1.U3RXDP1; no longer D5.D2-, IC1A.USB_SSRXP_DN1, J4USBA.STDA_SSRX+
- net USB1_SSTX_N: now also IC1G$1.U3TXDN1; no longer C64.2, D6.D1+, IC1A.USB_SSTXN_DN1
- net USB1_SSTX_P: now also IC1G$1.U3TXDP1; no longer C65.2, D6.D1-, IC1A.USB_SSTXP_DN1
- net USB2_DP_N: now also IC11.USB_DM, IC1G$1.U2DM2; no longer D6.D2+, IC1A.USB_DM_DN2, J5USBA.D-
- net USB2_DP_P: now also IC11.USB_DP, IC1G$1.U2DP2; no longer D6.D2-, IC1A.USB_DP_DN2, J5USBA.D+
- net USB2_SSRX_N: now also IC1G$1.U3RXDN2; no longer D7.D1+, IC1A.USB_SSRXN_DN2, J5USBA.STDA_SSRX-
- net USB2_SSRX_P: now also IC1G$1.U3RXDP2; no longer D7.D1-, IC1A.USB_SSRXP_DN2, J5USBA.STDA_SSRX+
- net USB2_SSTX_N: now also IC1G$1.U3TXDN2; no longer C68.2, D7.D2+, IC1A.USB_SSTXN_DN2
- net USB2_SSTX_P: now also IC1G$1.U3TXDP2; no longer C69.2, D7.D2-, IC1A.USB_SSTXP_DN2
- net USB3_DP_N: now also IC1G$1.U2DM3, R51.1; no longer D8.D1+, IC1A.USB_DM_DN3, J4USBB.D-
- net USB3_DP_P: now also IC1G$1.U2DP3, R52.2; no longer D8.D1-, IC1A.USB_DP_DN3, J4USBB.D+
- net USB3_SSRX_N: now also IC1G$1.U3RXDN3; no longer D8.D2+, IC1A.USB_SSRXN_DN3, J4USBB.STDA_SSRX-
- net USB3_SSRX_P: now also IC1G$1.U3RXDP3; no longer D8.D2-, IC1A.USB_SSRXP_DN3, J4USBB.STDA_SSRX+
- net USB3_SSTX_N: now also IC1G$1.U3TXDN3; no longer C72.2, D9.D1+, IC1A.USB_SSTXN_DN3
- net USB3_SSTX_P: now also IC1G$1.U3TXDP3; no longer C73.2, D9.D1-, IC1A.USB_SSTXP_DN3
- net USB4_DP_N: now also IC1G$1.U2DM4, J4.2; no longer D9.D2+, IC1A.USB_DM_DN4, J5USBB.D-
- net USB4_DP_P: now also IC1G$1.U2DP4, J4.3; no longer D9.D2-, IC1A.USB_DP_DN4, J5USBB.D+
- net USB4_SSRX_N: now also IC1G$1.U3RXDN4; no longer D10.D1+, IC1A.USB_SSRXN_DN4, J5USBB.STDA_SSRX-
- net USB4_SSRX_P: now also IC1G$1.U3RXDP4; no longer D10.D1-, IC1A.USB_SSRXP_DN4, J5USBB.STDA_SSRX+
- net USB4_SSTX_N: now also IC1G$1.U3TXDN4; no longer C76.2, D10.D2+, IC1A.USB_SSTXN_DN4
- net USB4_SSTX_P: now also IC1G$1.U3TXDP4; no longer C77.2, D10.D2-, IC1A.USB_SSTXP_DN4
Other:
- note added: "+3.3V LDO"
- note added: "5V │ R1 = 10k │ ●─── Vout (buffered) │ R2 = 22k (T1 → 2.5V) │ R3 = 10k (T2 → 1.8V) │ GND"
- note added: "CY7C68013A"
- note added: "DOWNSTREAM PORT1 - LOGIC ANALYSER"
- note added: "DOWNSTREAM PORT2 - FT4222 JTAG-SPI-I2C"
- note added: "DOWNSTREAM PORT2 - LOGIC LEVEL TRANSLATOR"
- note added: "DOWNSTREAM PORT3 - SWD PROGRAMMER/DEBUGGER"
- note added: "EEPROM"
- note added: "LOGIC LEVEL BUFFER CH0-7"
- note added: "LOGIC LEVEL BUFFER CH8-15"
- note added: "POWER"
- note added: "VCCA ≤ VCCB"
- note added: "VRERF_LOGIC = 1.8V V_COMP = ~1.5V"
- note added: "VRERF_LOGIC = 2.5V V_COMP = ~2.2V"
- note added: "VRERF_LOGIC = 3.3V V_COMP = ~3V"
- note removed: "DOWNSTREAM PORTS"
- note removed: "JUMPER J1 FOR NO WAKE SUPPORT"
- note removed: "POPULATE PULLDOWN IF I2C EEPROM NOT USED AND DO NOT POPULATE PULLUP"
- note removed: "POPULATE R1 FOR WAKE SUPPORT"
